File: wo33a/wo33a.sch (KiCad schematic (older format))
At the start: 77 parts, among them SW1 VRANGE, T1 232900-1

Commit message: moar work
Parts:
- removed R11: 1M, symbol Device:R_Variable_US
- removed R27: 5K, symbol Device:R_Variable_US
- added C19, C20: .05uf, symbol Device:CP1
- added C21, C22: 0.02uf, symbol Device:CP1
- added EXT.SYNC/H_INPUT: Conn_01x01_Female, symbol Connector:Conn_01x01_Female
- added L2, L3: 36uH, symbol Device:L
- added R33, R38: 1M, symbol Device:R_US
- added R34, R37: 820K, symbol Device:R_US
- added R35, RV11: 1M, symbol Device:R_POT_TRIM_US
- added R36: 1.2M, symbol Device:R_US
- added R68: 100K, symbol Device:R_POT_TRIM_US
- added R69: 180K, symbol Device:R_US
- added R? (x2): 10K, symbol Device:R_US
- added RV27: 5K, symbol Device:R_POT_TRIM_US
- added SW3: SW_DPDT_x2, symbol Switch:SW_DPDT_x2
- added TP? (x4): 220v, symbol Connector:TestPoint
- added V7: 3AQP, symbol wo33a:3AQP
Connections:
- net A1: now also SW3.4 (A)
- net B1: now also C21.1
- net GND: now also R36.1, R69.1, SW3.1 (A)
- net X1: now reaches T1.GRN (S2A)
- net X1: now also V7.1 (HTR)
- net X2: now reaches T1.GRN-YEL (S2B)
- net X2: now also V7.12 (HTR)
- net HumBalance: now reaches C13.1, R14.1, TP?.1, V1.8 (K_G3)
- net at R66.1, SW1.1, SW1.2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: now also RV11.1, RV11.2
- net at R31.1, TP?.1, V2.6 (A): now also L2.1, R?.2
- net at R29.1, TP?.1, V2.8 (K): now also RV27.1
- net at R12.1: now also RV11.3
- net at R22.1, R24.2, R32.2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: now also R34.1, R37.2, R68.1
- net at R28.1, TP?.1, V2.3 (K): now also RV27.2, RV27.3
- net at R25.1, TP?.1, V2.1 (A): now also L3.2, R?.1
- new net: C19.2, R33.2, TP?.1, V7.6 (D3)
- new net: C20.2, R38.1, V7.7 (D4)
- new net: R68.2, V7.8 (G2)
- new net: TP?.1, V7.9 (D1)
- new net: C19.1, L2.2, R?.1
- new net: C20.1, L3.1, R?.2
- new net: R33.1, R34.2, R35.1
- new net: R35.3, R37.1, R38.2
- new net: R35.2, R36.2
- new net: R68.3, R69.2
- new net: C21.2, SW3.3 (C)
- new net: C22.1, SW3.5 (B)
Other:
- note added: "Astigmatism\nAdjust"
- note added: "EXT"
- note added: "INT"
- note added: "V POS"
- moved on the sheet: T1, TP?
